File: pcb/VejasAuth.kicad_pcb (KiCad board)
At the start: 2 copper layers, 18.2 x 45.5 mm, 34 parts, among them J1 USB_A, J3 UP20-C-F-G-FL-P12-TR, SW3 PTS815 SJM 250 SMTR LFS, SW4 PTS815 SJM 250 SMTR LFS, U2 W25Q128JVS, U3 XC6206P332MR-G, U4 RP2350A-QFN60, Y1 ABM8-272-T3

Commit message: pcb1.1
Parts:
- moved U2 4.68 mm to (158.5, 95.4), turned to 90 degrees
- moved C21 1.96 mm to (168.8, 98.1)
- moved L1 1.96 mm to (169.8, 98.1)
- moved C20 1.94 mm to (167.7, 98.1)
- moved R1 1.86 mm to (157.4, 101.7)
- moved C3 1.85 mm to (157.4, 105.0)
- moved C2 1.85 mm to (157.4, 103.0)
- moved C6 1.85 mm to (157.4, 107.0)
- moved C10 1.41 mm to (167.5, 110.7)
- moved C13 1.41 mm to (161.2, 111.1)
- moved C14 1.41 mm to (168.8, 102.4)
- moved C16 1.41 mm to (162.7, 111.1)
- moved C4 1.41 mm to (168.8, 105.1)
- moved C5 1.41 mm to (164.2, 111.1)
- moved C8 1.41 mm to (168.8, 106.2)
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Routing:
- net GND: track 78.8 -> 46.0 mm, vias 9 -> 12
- net /QSPI_SS: track 18.0 -> 8.58 mm
- net +3V3: track 82.9 -> 90.5 mm, vias 3 -> 4
- net /QSPI_SD1: track 13.7 -> 6.74 mm
- net /QSPI_SD2: track 12.3 -> 5.40 mm
- net +1V1: track 31.7 -> 38.2 mm
- net /D+: track 48.0 -> 52.8 mm, vias 3 -> 2
- net /D-: track 50.6 -> 55.0 mm, vias 3 -> 4
- net /QSPI_SCLK: track 18.3 -> 15.3 mm
- net VBUS: track 50.8 -> 53.5 mm
- net Net-(U4-VREG_LX): track 4.20 -> 6.74 mm
- net Net-(R1-Pad2): track 18.8 -> 20.3 mm
- net /RUN: track 12.1 -> 13.5 mm
- net /QSPI_SD3: track 19.4 -> 20.5 mm
- net Net-(J3-CC1): track 2.01 -> 2.82 mm
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Other:
- board size 18.2 x 45.5 mm -> 16.9 x 45.5 mm

Commit message: pcb1.1.1
Parts:
- moved Y1 1.19 mm to (163.7, 117.0)
- moved SW3 1.19 mm to (159.2, 115.7)
- moved SW4 1.19 mm to (168.2, 115.7)
Routing:
- net VBUS: track 53.5 -> 52.2 mm
- net /RUN: track 13.5 -> 12.5 mm
- net Net-(R1-Pad2): track 20.3 -> 19.4 mm
Changed lines of the file:
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@@
 	(footprint "Crystal:Crystal_SMD_3225-4Pin_3.2x2.5mm"
 		(layer "F.Cu")
-		(at 164.8714 117.1854)
+		(at 163.703 116.967)
 		(descr "SMD3225/4, Crystal, 3.2x2.5mm package, SMD, generated with kicad-footprint-generator make_crystal.py, http://www.txccrystal.com/images/pdf/7m-accuracy.pdf")
 		(property "Reference" "Y1"
@@
 	(footprint "PTS815SJM250SMTRLFS:SW4_PTS815 SJM 250 SMTR LFS_CNK"
 		(layer "F.Cu")
-		(at 169.3926 115.951 -90)
+		(at 168.2242 115.7326 -90)
 		(tags "PTS815 SJM 250 SMTR LFS ")
 		(property "Reference" "SW4"
@@
 	(footprint "PTS815SJM250SMTRLFS:SW4_PTS815 SJM 250 SMTR LFS_CNK"
 		(layer "F.Cu")
-		(at 160.3756 115.951 -90)
+		(at 159.2072 115.7326 -90)
 		(tags "PTS815 SJM 250 SMTR LFS ")
 		(property "Reference" "SW3"
@@
 	)
 	(segment
-		(start 163.7714 114.7748)
-		(end 163.2712 114.2746)
-		(width 0.2)
-		(layer "F.Cu")
-		(net 2)
-	)
-	(segment
 		(start 165.7988 86.3186)
 		(end 167.4062 84.7112)
@@
 	)
 	(segment
-		(start 163.7714 116.3354)
-		(end 163.7714 114.7748)
-		(width 0.2)
-		(layer "F.Cu")
-		(net 2)
-	)
-	(segment
 		(start 165.7988 88.2018)
 		(end 166.4208 88.8238)
@@
 	)
 	(segment
+		(start 163.2712 114.3508)
+		(end 162.603 115.019)
+		(width 0.2)
+		(layer "F.Cu")
+		(net 2)
+	)
+	(segment
+		(start 163.2712 114.2746)
+		(end 163.2712 114.3508)
+		(width 0.2)
+		(layer "F.Cu")
+		(net 2)
+	)
+	(segment
 		(start 164.1945 111.9975)
 		(end 164.8206 112.6236)
@@
 	)
 	(segment
+		(start 162.603 115.019)
+		(end 162.603 116.117)
+		(width 0.2)
+		(layer "F.Cu")
+		(net 2)
+	)
+	(segment
 		(start 166.455608 101.2729)
 		(end 165.8579 101.870608)
@@
 	)
 	(via
-		(at 170.6372 89.281)
+		(at 170.053 91.948)
 		(size 0.6)
 		(drill 0.3)
@@
 	)
 	(segment
-		(start 166.7002 120.8532)
-		(end 171.202 116.3514)
+		(start 166.7002 120.8936)
+		(end 166.7002 120.8532)
 		(width 0.2)
 		(layer "B.Cu")
@@
 	)
 	(segment
-		(start 167.9956 90.3224)
-		(end 165.4302 90.3224)
+		(start 165.4302 90.3224)
+		(end 164.2364 89.1286)
 		(width 0.2)
 		(layer "B.Cu")
@@
 	)
 	(segment
-		(start 171.202 93.5288)
-		(end 167.9956 90.3224)
+		(start 166.7002 120.8532)
+		(end 171.202 116.3514)
 		(width 0.2)
 		(layer "B.Cu")
@@
 	)
 	(segment
-		(start 165.4302 90.3224)
-		(end 164.2364 89.1286)
+		(start 171.202 95.7386)
+		(end 165.7858 90.3224)
 		(width 0.2)
 		(layer "B.Cu")
@@
 	)
 	(segment
-		(start 166.7002 120.8936)
-		(end 166.7002 120.8532)
+		(start 171.202 116.3514)
+		(end 171.202 95.7386)
 		(width 0.2)
 		(layer "B.Cu")
@@
 	)
 	(segment
-		(start 171.202 116.3514)
-		(end 171.202 93.5288)
+		(start 165.7858 90.3224)
+		(end 165.4302 90.3224)
 		(width 0.2)
 		(layer "B.Cu")
@@
 	)
 	(segment
-		(start 170.467599 113.700999)
-		(end 169.2378 112.4712)
-		(width 0.2)
-		(layer "F.Cu")
-		(net 42)
-	)
-	(segment
 		(start 164.6579 110.17085)
 		(end 164.6579 109.2686)
@@
 	)
 	(segment
-		(start 169.2378 112.4712)
+		(start 168.7322 112.4712)
 		(end 165.5915 112.4712)
 		(width 0.2)
@@
 	)
 	(segment
-		(start 170.467599 118.201001)
-		(end 170.467599 113.700999)
+		(start 169.299199 113.482599)
+		(end 169.299199 113.038199)
+		(width 0.2)
+		(layer "F.Cu")
+		(net 42)
+	)
+	(segment
+		(start 169.299199 117.982601)
+		(end 169.299199 113.482599)
+		(width 0.2)
+		(layer "F.Cu")
+		(net 42)
+	)
+	(segment
+		(start 169.299199 113.038199)
+		(end 168.7322 112.4712)
 		(width 0.2)
 		(layer "F.Cu")
@@
 	)
 	(segment
-		(start 162.5092 113.455043)
-		(end 162.5092 116.7732)
+		(start 162.603 117.817)
+		(end 161.5694 116.7834)
 		(width 0.2)
 		(layer "F.Cu")
@@
 	)
 	(segment
-		(start 161.8337 111.5326)
-		(end 161.8337 112.779543)
+		(start 162.6579 110.5816)
+		(end 162.7213 110.645)
 		(width 0.2)
 		(layer "F.Cu")
@@
 	)
 	(segment
-		(start 162.6579 110.5816)
-		(end 162.7213 110.645)
+		(start 161.8337 112.779543)
+		(end 161.8337 111.5326)
 		(width 0.2)
 		(layer "F.Cu")
@@
 	)
 	(segment
-		(start 162.6579 109.2686)
-		(end 162.6579 110.5816)
+		(start 161.5694 113.043843)
+		(end 161.8337 112.779543)
 		(width 0.2)
 		(layer "F.Cu")
@@
 	)
 	(segment
-		(start 161.8337 112.779543)
-		(end 162.5092 113.455043)
+		(start 161.8337 111.5326)
+		(end 162.7213 110.645)
 		(width 0.2)
 		(layer "F.Cu")
@@
 	)
 	(segment
-		(start 162.7213 110.645)
-		(end 161.8337 111.5326)
+		(start 162.6579 109.2686)
+		(end 162.6579 110.5816)
 		(width 0.2)
 		(layer "F.Cu")
@@
 	)
 	(segment
-		(start 162.5092 116.7732)
-		(end 163.7714 118.0354)
+		(start 161.5694 116.7834)
+		(end 161.5694 113.043843)
 		(width 0.2)
 		(layer "F.Cu")
@@
 	)
 	(segment
-		(start 165.608 114.6022)
-		(end 165.608 116.3124)
+		(start 164.5412 115.8552)
+		(end 164.803 116.117)
 		(width 0.2)
 		(layer "F.Cu")
@@
 	)
 	(segment
-		(start 165.608 116.3124)
-		(end 165.6158 116.3202)
+		(start 164.5412 114.6068)
+		(end 164.5412 115.8552)
 		(width 0.2)
 		(layer "F.Cu")
@@
 	)
 	(segment
-		(start 161.450599 113.700999)
-		(end 161.450599 118.201001)
+		(start 160.282199 117.982601)
+		(end 160.282199 113.482599)
 		(width 0.2)
 		(layer "F.Cu")
@@
 	)
 	(segment
-		(start 161.450599 113.700999)
-		(end 160.350599 113.700999)
-		(width 0.2)
-		(layer "F.Cu")
-		(net 57)
-	)
-	(segment
 		(start 156.2141 101.9302)
 		(end 156.4427 101.7016)
@@
 	)
 	(segment
-		(start 160.0276 112.913443)
-		(end 158.874157 111.76)
+		(start 160.282199 113.482599)
+		(end 160.282199 113.168042)
 		(width 0.2)
 		(layer "F.Cu")
@@
 	)
 	(segment
-		(start 160.0276 113.378)
-		(end 160.0276 112.913443)
+		(start 160.282199 113.168042)
+		(end 158.874157 111.76)
 		(width 0.2)
 		(layer "F.Cu")

Commit message: idk
Parts:
- added D1: WS2812B-2020, LED_SMD:LED_WS2812B-2020_PLCC4_2.0x2.0mm, F.Cu at (169.6, 89.0)
- added D2: D, Diode_SMD:D_0402_1005Metric, F.Cu at (168.6, 91.4)
Connections:
- U4 pad 31: unconnected-(U4-GPIO19-Pad31) -> /LED
Routing:
- net /LED: track 0.00 -> 22.5 mm, vias 0 -> 2
- net VBUS: track 52.2 -> 54.3 mm, vias 2 -> 3
- net /QSPI_SD0: track 13.1 -> 11.4 mm
- net Net-(D1-VSS): track 0.00 -> 1.41 mm
- net GND: track 45.9 -> 44.5 mm, vias 12 -> 13
- net +3V3: track 90.5 -> 89.2 mm
- net /QSPI_SD3: track 20.5 -> 19.9 mm

Commit message: pcb
Parts:
- added REF**: MountingHole_2.2mm_M2, MountingHole:MountingHole_2.2mm_M2, F.Cu at (169.6, 122.2)
- moved J3 2.42 mm to (161.3, 124.7)
Routing:
- net VBUS: track 54.3 -> 59.2 mm
- net GND: track 44.5 -> 40.5 mm
- net /D+: track 52.6 -> 55.1 mm
- net Net-(J3-CC1): track 2.82 -> 5.19 mm
- net /D-: track 55.0 -> 57.2 mm
- net /QSPI_SD2: track 5.40 -> 4.81 mm
Other:
- board text added: "A C T I O N"
- board text added: "My personal Yubikey clone!"
- board text added: "R E S E T"
- board text added: "VejasAuth"
- board text added: "made by vejas, October 2025"

Commit message: pcb
Parts:
- added G***: LOGO, LOGO, F.Cu at (167.1, 93.9)
- added R6: 33, Resistor_SMD:R_0402_1005Metric, F.Cu at (168.8, 101.3)
- C21: value C -> 4.7uF
- L1: footprint Inductor_SMD:L_0402_1005Metric -> Inductor_SMD:L_0805_2012Metric
- moved C12 2.57 mm to (168.7, 98.1), turned to 90 degrees
- moved C21 2.25 mm to (169.0, 100.3), turned to 0 degrees
- moved D1 0.57 mm to (169.4, 88.4), turned to 180 degrees
- moved L1 0.53 mm to (170.4, 97.9)
- renumbered SW3 to SW1, SW4 to SW2
Connections:
- C21 pad 1: +3V3 -> Net-(U4-VREG_AVDD)
- D1 pad 2: Net-(D1-VSS) -> GND
- D1 pad 4: GND -> Net-(D1-VDD)
- D2 pad 1: Net-(D1-VSS) -> Net-(D1-VDD)
- U4 pad 46: +3V3 -> Net-(U4-VREG_AVDD)
Routing:
- net Net-(U4-VREG_AVDD): track 0.00 -> 3.53 mm
- net /LED: track 22.5 -> 25.8 mm
- net +3V3: track 89.2 -> 86.7 mm
- net Net-(D1-VDD): track 0.00 -> 1.95 mm
- net Net-(D1-VSS): track 1.41 -> 0.00 mm
- net GND: track 40.5 -> 41.1 mm, vias 13 -> 12

Commit message: cool stuff V1 i think
Parts:
- removed D2: D, Diode_SMD:D_0402_1005Metric
- SW1, SW2: value PTS815 SJM 250 SMTR LFS -> SW_SPST; footprint PTS815SJM250SMTRLFS:SW4_PTS815 SJM 250 SMTR LFS_CNK -> Button_Switch_SMD:SW_Push_SPST_NO_Alps_SKRK
- moved SW1 0.46 mm to (159.7, 115.7)
- moved SW2 0.36 mm to (167.9, 115.7)
Connections:
- D1 pad 4: Net-(D1-VDD) -> VBUS
- R1 pad 2: Net-(R1-Pad2) -> Net-(SW1-A)
- SW1 pad 1: Net-(R1-Pad2) -> Net-(SW1-A)
- SW1 pad 2: Net-(R1-Pad2) -> GND
- SW2 pad 2: /RUN -> GND
Routing:
- net Net-(R1-Pad2): track 19.0 -> 0.00 mm
- net Net-(SW1-A): track 0.00 -> 13.9 mm
- net /RUN: track 12.5 -> 6.35 mm
- net VBUS: track 59.2 -> 62.2 mm
- net Net-(D1-VDD): track 1.95 -> 0.00 mm
- net GND: track 41.1 -> 42.5 mm

Commit message: big update
Parts:
- removed J1: USB_A, Connector_USB:USB_A_Molex_48037-2200_Horizontal
- added J2: USB_C_Receptacle_USB2.0_16P, Connector_USB:USB_C_Receptacle_GCT_USB4105-xx-A_16P_TopMnt_Horizontal, F.Cu at (161.3, 127.0)
- added R7: 5.1k, Resistor_SMD:R_0402_1005Metric, F.Cu at (160.0, 121.2)
- J3: value UP20-C-F-G-FL-P12-TR -> UP2-AH-4-TH; footprint footprint:SAMESKY_UP20-C-F-G-FL-P12-TR -> usb a tht:CUI_UP2-AH-4-TH
- moved J3 42.8 mm to (163.6, 82.0), turned to 180 degrees
- moved REF** 3.87 mm to (169.3, 126.1)
- moved R2 1.49 mm to (163.1, 121.2), turned to 90 degrees
Connections:
- R2 pad 1: Net-(J3-CC1) -> Net-(J2-CC2)
Routing:
- net Net-(J3-CC1): track 5.28 -> 0.00 mm
- net GND: track 42.5 -> 38.9 mm, vias 12 -> 16
- net Net-(J2-CC2): track 0.00 -> 1.62 mm
- net Net-(J2-CC1): track 0.00 -> 1.62 mm
- net VBUS: track 62.2 -> 63.3 mm
- net /D-: track 57.2 -> 57.7 mm
Other:
- board size 16.9 x 45.5 mm -> 16.9 x 51.3 mm
