File: pcb/VejasAuth.kicad_sch (KiCad schematic)
At the start: 19 parts, among them U1 RP2040, U2 W25Q128JVSIQ, Y1 12MHz

Commit message: schem
Parts:
- removed U1: RP2040, Package_DFN_QFN:QFN-56-1EP_7x7mm_P0.4mm_EP3.2x3.2mm, symbol MCU_RaspberryPi:RP2040
- added C16, C17: 22pF, symbol Device:C
- added C18, C19: 10uF, symbol Device:C
- added C20: 4.7uF, symbol Device:C
- added C21: C, symbol Device:C
- added J1: USB_A, symbol Connector:USB_A
- added L1: 3.3uF, symbol Device:L
- added P1: USB_C_Plug_USB2.0, symbol Connector:USB_C_Plug_USB2.0
- added R3: 1k, symbol Device:R
- added R4, R5: 27, symbol Device:R
- added R6: 5.1k, symbol Device:R
- added SW1, SW2: C720477, symbol Switch:SW_SPST
- added U3: XC6206P332MR-G, Package_TO_SOT_SMD:SOT-23-3, symbol Regulator_Linear:XC6206PxxxMR
- added U4: RP2350A-QFN60, symbol RP2035:RP2350A-QFN60
- C1: value 2.2uF -> 4.7uF
- C3: value 1uF -> 100nF
- C4: value 100nF -> 4.7uF
- R1: value 27 -> 1k
- R2: value 27 -> 5.1k
- U2: value W25Q128JVSIQ -> W25Q128JVS
- Y1: value 12MHz -> ABM8-272-T3
Connections:
- net 3V3 is gone; now on net +3V3: C2.1, U2.8 (VCC)
- net +1V1: now also C20.1, L1.1, U4.23 (DVDD), U4.39 (DVDD), U4.50 (VREG_FB), U4.6 (DVDD)
- net +3V3: now also C1.1, C19.1, C21.1, U3.2 (VO), U4.1 (IOVDD), U4.11 (IOVDD), U4.20 (IOVDD), U4.30 (IOVDD), U4.38 (IOVDD), U4.44 (ADC_AVDD), U4.45 (IOVDD), U4.46 (VREG_AVDD), U4.49 (VREG_VIN), U4.53 (USB_OTP_VDD), U4.54 (QSPI_IOVDD)
- net D+: now also J1.3 (D+), P1.A6 (D+), R4.1; no longer R1.1
- net D-: now also J1.2 (D-), P1.A7 (D-), R5.1; no longer R2.1
- net GND: now also C1.2, R2.2, U2.4 (GND), Y1.2, Y1.4, C16.1, C17.1, C18.2, C19.2, C20.2, C21.2, J1.4 (GND), J1.5 (Shield), P1.A1 (GND), P1.A12 (GND), P1.B1 (GND), P1.B12 (GND), P1.S1 (SHIELD), R6.2, SW1.2 (B), SW2.2 (B), U3.1 (GND), U4.47 (VREG_PGND), U4.61 (GND); no longer C1.1
- net QSPI_SCLK: now also U4.56 (QSPI_SCLK)
- net QSPI_SD0: now also U4.57 (QSPI_SD0)
- net QSPI_SD1: now also U4.59 (QSPI_SD1)
- net QSPI_SD2: now also U4.58 (QSPI_SD2)
- net QSPI_SD3: now also U4.55 (QSPI_SD3)
- net QSPI_SS: now also R1.1, U4.60 (QSPI_SS)
- net RUN: now also SW2.1 (A), U4.26 (RUN)
- net XIN: now also Y1.1, C16.2, U4.21 (XIN)
- net XOUT: now also R3.2, U4.22 (XOUT)
- net at R1.2: now also SW1.1 (A)
- net at Y1.3: now also C17.2, R3.1
- new net: R4.2, U4.52 (USB_DP)
- new net: P1.A5 (CC), R2.1
- new net: L1.2, U4.48 (VREG_LX)
- new net: R5.2, U4.51 (USB_DM)
- new net: P1.B5 (VCONN), R6.1
- new net VBUS: C18.1, J1.1 (VBUS), P1.A4 (VBUS), P1.A9 (VBUS), P1.B4 (VBUS), P1.B9 (VBUS), U3.3 (VI)
Other:
- moved on the sheet: C10, C11, C12, C13, C14, C2, C3, C4, C5, C6, C7, C8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

Commit message: pcb1.0
Parts:
- removed P1: USB_C_Plug_USB2.0, symbol Connector:USB_C_Plug_USB2.0
- removed R6: 5.1k, symbol Device:R
- removed SW1, SW2: C720477, symbol Switch:SW_SPST
- added J2: Conn_01x05_Pin, symbol Connector:Conn_01x05_Pin
- added J3: UP20-C-F-G-FL-P12-TR, footprint:SAMESKY_UP20-C-F-G-FL-P12-TR, symbol usbc:UP20-C-F-G-FL-P12-TR
- added SW3, SW4: PTS815 SJM 250 SMTR LFS, PTS815SJM250SMTRLFS:SW4_PTS815 SJM 250 SMTR LFS_CNK, symbol PTS815SJM250SMTRLFS:PTS815_SJM_250_SMTR_LFS
- C1, C10, C11, C12, C13, C14, C16, C17, C2, C20, C21, C3, C4, C5, C6, C8, C9: footprint (none) -> Capacitor_SMD:C_0402_1005Metric
- C18, C19, C7: footprint (none) -> Capacitor_SMD:C_0603_1608Metric
- J1: footprint (none) -> Connector_USB:USB_A_Molex_48037-2200_Horizontal
- L1: value 3.3uF -> 3.3u; footprint (none) -> Inductor_SMD:L_0402_1005Metric
- R1, R2, R3, R4, R5: footprint (none) -> Resistor_SMD:R_0402_1005Metric
- U4: footprint (none) -> Package_DFN_QFN:QFN-60-1EP_7x7mm_P0.4mm_EP3.4x3.4mm_ThermalVias
Connections:
- net D+: now also J3.A6 (DP1)
- net D-: now also J3.A7 (DN1)
- net GND: now also J3.A1 (GND), J3.A12 (GND__1), J3.B12 (GND__2), J3.SH1 (SHIELD), J3.SH2 (SHIELD__1), SW3.3, SW3.4, SW4.3, SW4.4
- net RUN: now also SW4.1, SW4.2
- net VBUS: now also J3.A4 (VBUS), J3.B9 (VBUS__1)
- net at R1.2: now also SW3.1, SW3.2
- net at R2.1: now also J3.A5 (CC1)
- no-connect marks 0 -> 4
Other:
- moved on the sheet: R1, R2

Commit message: idk
Parts:
- added D1: WS2812B-2020, LED_SMD:LED_WS2812B-2020_PLCC4_2.0x2.0mm, symbol LED:WS2812B-2020
- added D2: D, Diode_SMD:D_0402_1005Metric, symbol Device:D
Connections:
- net GND: now also D1.4 (VDD)
- net VBUS: now also D2.2 (A)
- net LED: now reaches U4.31 (GPIO19)
- net LED: now also D1.3 (DIN)
- new net: D1.2 (VSS), D2.1 (K)
- no-connect marks 4 -> 5
Other:
- note added: "VSS means Voltage at Source VDD means Voltage at Drain"

Commit message: pcb
Parts:
- removed J2: Conn_01x05_Pin, symbol Connector:Conn_01x05_Pin
- added R6: 33, Resistor_SMD:R_0402_1005Metric, symbol Device:R
- C21: value C -> 4.7uF
- L1: footprint Inductor_SMD:L_0402_1005Metric -> Inductor_SMD:L_0805_2012Metric
- renumbered SW3 to SW1, SW4 to SW2
Connections:
- net +3V3: now also R6.1; no longer C21.1, U4.46 (VREG_AVDD)
- net GND: now also D1.2 (VSS); no longer D1.4 (VDD)
- net at D2.1 (K): now also D1.4 (VDD); no longer D1.2 (VSS)
- new net: C21.1, R6.2, U4.46 (VREG_AVDD)
Other:
- moved on the sheet: D1, D2
Changed lines of the file:
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@@
 	)
 	(no_connect
-		(at 309.88 132.08)
+		(at 325.12 132.08)
 	)
 	(no_connect
@@
 	(wire
 		(pts
-			(xy 317.5 116.84) (xy 317.5 113.03)
+			(xy 317.5 115.57) (xy 317.5 113.03)
 		)
 		(stroke
@@
 	(wire
 		(pts
+			(xy 317.5 123.19) (xy 317.5 124.46)
+		)
+		(stroke
+			(width 0)
+			(type default)
+		)
+	)
+	(wire
+		(pts
 			(xy 114.3 57.15) (xy 118.11 57.15)
 		)
@@
 	(wire
 		(pts
-			(xy 332.74 132.08) (xy 325.12 132.08)
+			(xy 302.26 132.08) (xy 309.88 132.08)
 		)
 		(stroke
@@
 	(wire
 		(pts
+			(xy 46.99 62.23) (xy 63.5 62.23)
+		)
+		(stroke
+			(width 0)
+			(type default)
+		)
+	)
+	(wire
+		(pts
 			(xy 63.5 69.85) (xy 63.5 71.12)
 		)
@@
 	(wire
 		(pts
-			(xy 22.86 62.23) (xy 63.5 62.23)
+			(xy 22.86 62.23) (xy 39.37 62.23)
 		)
 		(stroke
@@
 	)
 	(label "LED"
-		(at 332.74 132.08 180)
+		(at 302.26 132.08 0)
 		(effects
 			(font
 				(size 1.27 1.27)
 			)
-			(justify right bottom)
+			(justify left bottom)
 		)
 	)
@@
 	(symbol
 		(lib_id "Device:R")
+		(at 43.18 62.23 90)
+		(unit 1)
+		(exclude_from_sim no)
+		(in_bom yes)
+		(on_board yes)
+		(dnp no)
+		(fields_autoplaced yes)
+		(property "Reference" "R6"
+			(at 43.18 55.88 90)
+			(effects
+				(font
+					(size 1.27 1.27)
+				)
+			)
+		)
+		(property "Value" "33"
+			(at 43.18 58.42 90)
+			(effects
+				(font
+					(size 1.27 1.27)
+				)
+			)
+		)
+		(property "Footprint" "Resistor_SMD:R_0402_1005Metric"
+			(at 43.18 64.008 90)
+			(effects
+				(font
+					(size 1.27 1.27)
+				)
+				(hide yes)
+			)
+		)
+		(property "Datasheet" "~"
+			(at 43.18 62.23 0)
+			(effects
+				(font
+					(size 1.27 1.27)
+				)
+				(hide yes)
+			)
+		)
+		(property "Description" "Resistor"
+			(at 43.18 62.23 0)
+			(effects
+				(font
+					(size 1.27 1.27)
+				)
+				(hide yes)
+			)
+		)
+		(pin "2"
+		)
+		(pin "1"
+		)
+		(instances
+			(project ""
+				(path "/4e910406-fdd9-4bd9-bcc6-3116971ff91a"
+					(reference "R6")
+					(unit 1)
+				)
+			)
+		)
+	)
+	(symbol
+		(lib_id "Device:R")
 		(at 138.43 73.66 270)
 		(mirror x)
@@
 	(symbol
 		(lib_id "LED:WS2812B-2020")
-		(at 317.5 132.08 180)
+		(at 317.5 132.08 0)
 		(unit 1)
 		(exclude_from_sim no)
@@
 		(fields_autoplaced yes)
 		(property "Reference" "D1"
-			(at 331.47 126.6346 0)
+			(at 331.47 125.6598 0)
 			(effects
 				(font
@@
 		)
 		(property "Value" "WS2812B-2020"
-			(at 331.47 129.1746 0)
+			(at 331.47 128.1998 0)
 			(effects
 				(font
@@
 		)
 		(property "Footprint" "LED_SMD:LED_WS2812B-2020_PLCC4_2.0x2.0mm"
-			(at 316.23 124.46 0)
+			(at 318.77 139.7 0)
 			(effects
 				(font
@@
 		)
 		(property "Datasheet" "https://cdn-shop.adafruit.com/product-files/4684/4684_WS2812B-2020_V1.3_EN.pdf"
-			(at 314.96 122.555 0)
+			(at 320.04 141.605 0)
 			(effects
 				(font
@@
 			)
 		)
-		(property "Footprint" "Inductor_SMD:L_0402_1005Metric"
+		(property "Footprint" "Inductor_SMD:L_0805_2012Metric"
 			(at 49.53 81.28 0)
 			(effects
@@
 		(dnp no)
 		(fields_autoplaced yes)
-		(property "Reference" "SW4"
+		(property "Reference" "SW2"
 			(at 347.98 68.58 0)
 			(effects
@@
 			(project ""
 				(path "/4e910406-fdd9-4bd9-bcc6-3116971ff91a"
-					(reference "SW4")
+					(reference "SW2")
 					(unit 1)
 				)
@@
 			)
 		)
-		(property "Value" "C"
+		(property "Value" "4.7uF"
 			(at 67.31 67.3099 0)
 			(effects
@@
 		(dnp no)
 		(fields_autoplaced yes)
-		(property "Reference" "SW3"
+		(property "Reference" "SW1"
 			(at 347.98 43.18 0)
 			(effects
@@
 			(project ""
 				(path "/4e910406-fdd9-4bd9-bcc6-3116971ff91a"
-					(reference "SW3")
+					(reference "SW1")
 					(unit 1)
 				)
@@
 	(symbol
 		(lib_id "Device:D")
-		(at 317.5 120.65 90)
+		(at 317.5 119.38 90)
 		(unit 1)
 		(exclude_from_sim no)
@@
 		(fields_autoplaced yes)
 		(property "Reference" "D2"
-			(at 320.04 119.3799 90)
+			(at 320.04 118.1099 90)
 			(effects
 				(font
@@
 		)
 		(property "Value" "D"
-			(at 320.04 121.9199 90)
+			(at 320.04 120.6499 90)
 			(effects
 				(font
@@
 		)
 		(property "Footprint" "Diode_SMD:D_0402_1005Metric"
-			(at 317.5 120.65 0)
+			(at 317.5 119.38 0)
 			(effects
 				(font
@@
 		)
 		(property "Datasheet" "~"
-			(at 317.5 120.65 0)
+			(at 317.5 119.38 0)
 			(effects
 				(font
@@
 		)
 		(property "Description" "Diode"
-			(at 317.5 120.65 0)
+			(at 317.5 119.38 0)
 			(effects
 				(font
@@
 		)
 		(property "Sim.Device" "D"
-			(at 317.5 120.65 0)
+			(at 317.5 119.38 0)
 			(effects
 				(font
@@
 		)
 		(property "Sim.Pins" "1=K 2=A"
-			(at 317.5 120.65 0)
+			(at 317.5 119.38 0)
 			(effects
 				(font
@@
 					(unit 1)
 				)
-			)
-		)
-	)
-	(symbol
-		(lib_id "Connector:Conn_01x05_Pin")
-		(at 157.48 57.15 0)
-		(unit 1)
-		(exclude_from_sim no)
-		(in_bom yes)
-		(on_board yes)
-		(dnp no)
-		(fields_autoplaced yes)
-		(property "Reference" "J2"
-			(at 158.115 46.99 0)
-			(effects
-				(font
-					(size 1.27 1.27)
-				)
-			)
-		)
-		(property "Value" "Conn_01x05_Pin"
-			(at 158.115 49.53 0)
-			(effects
-				(font
-					(size 1.27 1.27)
-				)
-			)
-		)
-		(property "Footprint" ""
-			(at 157.48 57.15 0)
-			(effects
-				(font
-					(size 1.27 1.27)
-				)
-				(hide yes)
-			)
-		)
-		(property "Datasheet" "~"
-			(at 157.48 57.15 0)
-			(effects
-				(font
-					(size 1.27 1.27)
-				)
-				(hide yes)
-			)
-		)
-		(property "Description" "Generic connector, single row, 01x05, script generated"
-			(at 157.48 57.15 0)
-			(effects
-				(font
-					(size 1.27 1.27)
-				)
-				(hide yes)
-			)
-		)
-		(pin "4"
-		)
-		(pin "5"
-		)
-		(pin "3"
-		)
-		(pin "2"
-		)
-		(pin "1"
-		)
-		(instances
-			(project ""
-				(path "/4e910406-fdd9-4bd9-bcc6-3116971ff91a"
-					(reference "J2")
-					(unit 1)
-				)

Commit message: cool stuff V1 i think
Parts:
- removed D2: D, Diode_SMD:D_0402_1005Metric, symbol Device:D
- removed SW1, SW2: PTS815 SJM 250 SMTR LFS, PTS815SJM250SMTRLFS:SW4_PTS815 SJM 250 SMTR LFS_CNK, symbol PTS815SJM250SMTRLFS:PTS815_SJM_250_SMTR_LFS
- added SW1, SW2: SW_SPST, Button_Switch_SMD:SW_Push_SPST_NO_Alps_SKRK, symbol Switch:SW_SPST
Connections:
- net GND: now also SW1.2 (B), SW2.2 (B)
- net RUN: now also SW2.1 (A)
- net VBUS: now also D1.4 (VDD)
- net at R1.2: now also SW1.1 (A)
Other:
- note removed: "VSS means Voltage at Source VDD means Voltage at Drain"
- moved on the sheet: R1

Commit message: big update
Parts:
- removed J1: USB_A, Connector_USB:USB_A_Molex_48037-2200_Horizontal, symbol Connector:USB_A
- removed J3: UP20-C-F-G-FL-P12-TR, footprint:SAMESKY_UP20-C-F-G-FL-P12-TR, symbol usbc:UP20-C-F-G-FL-P12-TR
- added J2: USB_C_Receptacle_USB2.0_16P, Connector_USB:USB_C_Receptacle_GCT_USB4105-xx-A_16P_TopMnt_Horizontal, symbol Connector:USB_C_Receptacle_USB2.0_16P
- added J3: UP2-AH-4-TH, usb a tht:CUI_UP2-AH-4-TH, symbol usb a tht:UP2-AH-4-TH
- added R7: 5.1k, Resistor_SMD:R_0402_1005Metric, symbol Device:R
Connections:
- net D+: now also J2.A6 (D+), J2.B6 (D+), J3.3 (D+)
- net D-: now also J2.A7 (D-), J2.B7 (D-), J3.2 (D-)
- net GND: now also J2.A1 (GND), J2.A12 (GND), J2.A8 (SBU1), J2.B1 (GND), J2.B12 (GND), J2.B8 (SBU2), J2.S1 (SHIELD), J3.4 (GND), J3.SH1 (SHIELD), J3.SH2 (SHIELD), R7.2
- net VBUS: now also J2.A4 (VBUS), J2.A9 (VBUS), J2.B4 (VBUS), J2.B9 (VBUS), J3.1 (VCC)
- net at R2.1: now also J2.B5 (CC2)
- new net: J2.A5 (CC1), R7.1
- no-connect marks 5 -> 1
Other:
- moved on the sheet: D1, R1, R2, SW1, SW2
